Commit message: motion dataset changed

File: reacher_simulate/xml/reacher_0.urdf (robot description, URDF)
Before this commit: robot pybullet_reacher_robot, 4 links, 3 joints
Links:
- added link link4, mass 1.0; collision sphere radius=0.02; visual sphere radius=0.02
- link link1: geometry collision cylinder length=0.10224867402000892 radius=0.015; visual cylinder length=0.10224867402000892 radius=0.015
- link link2: geometry collision cylinder length=0.3209705008435014 radius=0.015; visual cylinder length=0.3209705008435014 radius=0.015
- link link3: geometry collision cylinder length=0.16794280810859813 radius=0.015; visual cylinder length=0.16794280810859813 radius=0.015
Joints:
- added joint joint4: type revolute, parent link3, child link4, origin xyz=0.16794280810859813 0.0 0.0 rpy=0.0 -0.0 0.0, axis 0. 0. 1., limit lower=-2.96705 upper=2.96705 effort=300.0 velocity=200.0
- joint joint2: origin xyz=0.2977012539596089 0.0 0.0 rpy=0.0 -0.0 0.0 -> xyz=0.10224867402000892 0.0 0.0 rpy=0.0 -0.0 0.0
- joint joint3: origin xyz=0.1982327299845677 0.0 0.0 rpy=0.0 -0.0 0.0 -> xyz=0.3209705008435014 0.0 0.0 rpy=0.0 -0.0 0.0

File: reacher_simulate/xml/reacher_1.urdf (robot description, URDF)
Before this commit: robot pybullet_reacher_robot, 4 links, 3 joints
Links:
- link link1: geometry collision cylinder length=0.3802880911634623 radius=0.015; visual cylinder length=0.3802880911634623 radius=0.015
- link link2: geometry collision cylinder length=0.11987230741893898 radius=0.015; visual cylinder length=0.11987230741893898 radius=0.015
Joints:
- joint joint2: origin xyz=0.14986494815494844 0.0 0.0 rpy=0.0 -0.0 0.0 -> xyz=0.3802880911634623 0.0 0.0 rpy=0.0 -0.0 0.0
- joint joint3: origin xyz=0.20969656193487146 0.0 0.0 rpy=0.0 -0.0 0.0 -> xyz=0.11987230741893898 0.0 0.0 rpy=0.0 -0.0 0.0
