Commit message: simulate update

File: reacher_simulate/xml/reacher_infer.urdf (robot description, URDF)
Before this commit: robot pybullet_reacher_robot, 6 links, 5 joints
Links:
- link link1: geometry collision cylinder length=0.009180068969726562 radius=0.015; visual cylinder length=0.009180068969726562 radius=0.015
- link link2: geometry collision cylinder length=0.004108548164367676 radius=0.015; visual cylinder length=0.004108548164367676 radius=0.015
- link link3: geometry collision cylinder length=0.0027573108673095703 radius=0.015; visual cylinder length=0.0027573108673095703 radius=0.015
- link link4: geometry collision cylinder length=0.0009915828704833984 radius=0.015; visual cylinder length=0.0009915828704833984 radius=0.015
Joints:
- joint joint2: origin xyz=0.0 0.0 0.0 rpy=0.0 -0.0 0.0 -> xyz=0.009180068969726562 0.0 0.0 rpy=0.0 -0.0 0.0
- joint joint3: origin xyz=0.3406 0.0 0.0 rpy=0.0 -0.0 0.0 -> xyz=0.004108548164367676 0.0 0.0 rpy=0.0 -0.0 0.0
- joint joint4: origin xyz=0.2549 0.0 0.0 rpy=0.0 -0.0 0.0 -> xyz=0.0027573108673095703 0.0 0.0 rpy=0.0 -0.0 0.0
- joint joint5: origin xyz=0.3095 0.0 0.0 rpy=0.0 -0.0 0.0 -> xyz=0.0009915828704833984 0.0 0.0 rpy=0.0 -0.0 0.0
